Commit message: Add README

File: models/diff_drive/diff_drive.xacro (robot description, xacro)
@@ -3,8 +3,8 @@
 <robot name="diff_drive" xmlns:xacro="http://www.ros.org/wiki/xacro">
   <!-- Start by including all required xacro files which hold the macros -->
-  <xacro:include filename="$(find kobuki_lane)/models/diff_drive/diff_drive.gazebo" />
-  <xacro:include filename="$(find kobuki_lane)/models/diff_drive/materials.xacro"   />
-  <xacro:include filename="$(find kobuki_lane)/models/diff_drive/macros.xacro"      />
-  <xacro:include filename="$(find kobuki_lane)/models/diff_drive/parameter.xacro"   />
+  <xacro:include filename="$(find rosbot)/models/diff_drive/diff_drive.gazebo" />
+  <xacro:include filename="$(find rosbot)/models/diff_drive/materials.xacro"   />
+  <xacro:include filename="$(find rosbot)/models/diff_drive/macros.xacro"      />
+  <xacro:include filename="$(find rosbot)/models/diff_drive/parameter.xacro"   />
  <!-- Create a dummy link as base link -->
   <link name='base_link'>

File: models/diff_drive/parameter.xacro (robot description, xacro)
@@ -2,5 +2,5 @@
 <robot xmlns:xacro="http://www.ros.org/wiki/xacro">
   <!-- Load config file, TODO: Add more parameter -->
-  <xacro:property name="package" value="$(find kobuki_lane)"/>
+  <xacro:property name="package" value="$(find rosbot)"/>
   <xacro:property name="properties" value="${load_yaml(package + '/config/config.yaml')}"/>
   <!-- Define parameter for the differential drive robot -->
